File: src-kicad/peripherals.sch (KiCad schematic (older format))
At the start: 31 parts, among them J15 1x4_male_pin_Header_2.54mm, J16 1x4_male_pin_Header_2.54mm, J17 1x4_male_pin_Header_2.54mm, SW1 Switch, SW2 Switch, U7 ADS7924

Commit message: Kicad pcb migration: Capacitors C21, C26 and C30
Parts:
- C34, C35, C45, C46: footprint (none) -> Icezum:C_0402
Changed lines of the file:
@@
 F 0 "C46" V 8320 1970 50  0000 L CNN
 F 1 "100nF" V 8610 1960 50  0000 L CNN
-F 2 "" H 8488 1900 50  0000 C CNN
+F 2 "Icezum:C_0402" H 8488 1900 50  0001 C CNN
 F 3 "" H 8450 2050 50  0000 C CNN
 F 4 "X7R" V 8510 2170 50  0000 C CNN "Class"
@@
 F 0 "C45" V 8970 1970 50  0000 L CNN
 F 1 "100nF" V 9260 1960 50  0000 L CNN
-F 2 "" H 9138 1900 50  0000 C CNN
+F 2 "Icezum:C_0402" H 9138 1900 50  0001 C CNN
 F 3 "" H 9100 2050 50  0000 C CNN
 F 4 "X7R" V 9160 2170 50  0000 C CNN "Class"
@@
 F 0 "C34" H 3800 1420 50  0000 L CNN
 F 1 "100nF" H 3720 1630 50  0000 L CNN
-F 2 "" H 4088 1350 50  0000 C CNN
+F 2 "Icezum:C_0402" H 4088 1350 50  0001 C CNN
 F 3 "" H 4050 1500 50  0000 C CNN
 F 4 "X7R" H 3870 1490 50  0000 C CNN "Class"
@@
 F 0 "C35" H 3800 2320 50  0000 L CNN
 F 1 "100nF" H 3720 2530 50  0000 L CNN
-F 2 "" H 4088 2250 50  0000 C CNN
+F 2 "Icezum:C_0402" H 4088 2250 50  0001 C CNN
 F 3 "" H 4050 2400 50  0000 C CNN
 F 4 "X7R" H 3870 2390 50  0000 C CNN "Class"
@@
 B8 D2 A5 D0 D0 88 43 83 08 6C BD D2 A5 D0 D0 88 C3 36 11 89 E7 80 EE 2B 5D 12 0D 8D 28 1C 42 E0
 0D 11 99 76 E0 6E E0 E3 2B 5D 22 0D 8D 71 EC 07 1E E7 1B 7C F8 FF 01 FB D1 C8 6E 4C 03 14 F4 00
-00 00 00 49 45 4E 44 AE 42 60 82 00
+00 00 00 49 45 4E 44 AE 42 60 82 03
 EndData
 $EndBitmap

Commit message: Kicad pcb migration: More capacitors footprint assigned
Parts:
- C41: footprint (none) -> Icezum:C_0603
Changed lines of the file:
@@
 F 0 "C41" V 8320 1570 50  0000 L CNN
 F 1 "4.7uF" V 8610 1560 50  0000 L CNN
-F 2 "" H 8488 1500 50  0000 C CNN
+F 2 "Icezum:C_0603" H 8488 1500 50  0001 C CNN
 F 3 "" H 8450 1650 50  0000 C CNN
 F 4 "X5R" V 8510 1770 50  0000 C CNN "Class"

Commit message: Kicad pcb migration. R11 added. Some bug fixed in the schematics (R16 was missing)
Parts:
- R19, R20, R21: footprint (none) -> Icezum:R_0402
Changed lines of the file:
@@
 F 0 "R19" V 7830 1890 50  0000 C CNN
 F 1 "10R±5% 0.063w" V 7970 1950 39  0000 C CNN
-F 2 "" V 7830 2050 50  0000 C CNN
+F 2 "Icezum:R_0402" V 7830 2050 50  0001 C CNN
 F 3 "" H 7900 2050 50  0000 C CNN
 	1    7900 2050
@@
 F 0 "R20" V 9980 2340 50  0000 C CNN
 F 1 "10k±5% 0.063w" V 10120 2400 39  0000 C CNN
-F 2 "" V 9980 2500 50  0000 C CNN
+F 2 "Icezum:R_0402" V 9980 2500 50  0001 C CNN
 F 3 "" H 10050 2500 50  0000 C CNN
 	1    10050 2500
@@
 F 0 "R21" V 10230 2340 50  0000 C CNN
 F 1 "10k±5% 0.063w" V 10370 2400 39  0000 C CNN
-F 2 "" V 10230 2500 50  0000 C CNN
+F 2 "Icezum:R_0402" V 10230 2500 50  0001 C CNN
 F 3 "" H 10300 2500 50  0000 C CNN
 	1    10300 2500
@@
 F3 F0 1D 79 17 0B BC D0 AE 96 03 B8 3F 0C 6D B8 A2 A8 0B 16 2C 58 B0 60 C1 82 05 0B 16 2C 58 B0
 60 C1 82 05 0B 16 2C 58 B0 E0 7F 81 FF 00 64 C5 01 8A 14 5C 86 66 00 00 00 00 49 45 4E 44 AE 42
-60 82 E0
+60 82 39
 EndData
 $EndBitmap
