File: src-kicad/peripherals.sch (KiCad schematic (older format))
At the start: 31 parts, among them J15 1x4_male_pin_Header_2.54mm, J16 1x4_male_pin_Header_2.54mm, J17 1x4_male_pin_Header_2.54mm, SW1 Switch, SW2 Switch, U7 ADS7924

Commit message: migrated version V1.1 of Eeschema files
Parts:
- removed R17, R18: 270R±5% 0.0625w, Icezum:R_Array_Convex_4x0603, symbol Resistor_array_1x4
- removed SW1, SW2: Switch, Icezum:SW_SMD_60X3.8, symbol Switch
- added R17, R18, R40, R41, R42, R43, R44, R45: 2k2±5% 0.063w, symbol R
- added R31, R32: 10k±5% 0.0625w, symbol R
- added SW1, SW2: Switch, symbol Switch_4p
- LD0: renamed from D2; value Yellow -> Green
- LD1: renamed from D3; value Yellow -> Green
- LD2: renamed from D4; value Yellow -> Green
- LD3: renamed from D5; value Yellow -> Green
- LD4: renamed from D6; value Yellow -> Green
- LD5: renamed from D7; value Yellow -> Green
- LD6: renamed from D8; value Yellow -> Green
- LD7: renamed from D9; value Yellow -> Green
Connections:
- wire segments 80 -> 89
Other:
- moved on the sheet: C34, C35, C41, C45, C46

Commit message: se añaden huellas a los nuevos componentes y genera netlist
Parts:
- R17, R18, R31, R32, R40, R41, R42, R43, R44, R45: footprint (none) -> Icezum:R_0402
- SW1, SW2: footprint (none) -> Icezum:WE_434331013822_push_switch
Changed lines of the file:
@@
 F 0 "R18" V 1505 1450 50  0000 C CNN
 F 1 "2k2±5% 0.063w" V 1596 1450 50  0000 C CNN
-F 2 "" V 1630 1460 50  0000 C CNN
+F 2 "Icezum:R_0402" V 1630 1460 50  0001 C CNN
 F 3 "" H 1700 1460 50  0000 C CNN
 	1    1700 1600
@@
 F 0 "R17" V 1505 1050 50  0000 C CNN
 F 1 "2k2±5% 0.063w" V 1596 1050 50  0000 C CNN
-F 2 "" V 1630 1060 50  0000 C CNN
+F 2 "Icezum:R_0402" V 1630 1060 50  0001 C CNN
 F 3 "" H 1700 1060 50  0000 C CNN
 	1    1700 1200
@@
 F 0 "R40" V 1505 1850 50  0000 C CNN
 F 1 "2k2±5% 0.063w" V 1596 1850 50  0000 C CNN
-F 2 "" V 1630 1860 50  0000 C CNN
+F 2 "Icezum:R_0402" V 1630 1860 50  0001 C CNN
 F 3 "" H 1700 1860 50  0000 C CNN
 	1    1700 2000
@@
 F 0 "R41" V 1505 2250 50  0000 C CNN
 F 1 "2k2±5% 0.063w" V 1596 2250 50  0000 C CNN
-F 2 "" V 1630 2260 50  0000 C CNN
+F 2 "Icezum:R_0402" V 1630 2260 50  0001 C CNN
 F 3 "" H 1700 2260 50  0000 C CNN
 	1    1700 2400
@@
 F 0 "R42" V 1505 2650 50  0000 C CNN
 F 1 "2k2±5% 0.063w" V 1596 2650 50  0000 C CNN
-F 2 "" V 1630 2660 50  0000 C CNN
+F 2 "Icezum:R_0402" V 1630 2660 50  0001 C CNN
 F 3 "" H 1700 2660 50  0000 C CNN
 	1    1700 2800
@@
 F 0 "R43" V 1505 3050 50  0000 C CNN
 F 1 "2k2±5% 0.063w" V 1596 3050 50  0000 C CNN
-F 2 "" V 1630 3060 50  0000 C CNN
+F 2 "Icezum:R_0402" V 1630 3060 50  0001 C CNN
 F 3 "" H 1700 3060 50  0000 C CNN
 	1    1700 3200
@@
 F 0 "R44" V 1505 3450 50  0000 C CNN
 F 1 "2k2±5% 0.063w" V 1596 3450 50  0000 C CNN
-F 2 "" V 1630 3460 50  0000 C CNN
+F 2 "Icezum:R_0402" V 1630 3460 50  0001 C CNN
 F 3 "" H 1700 3460 50  0000 C CNN
 	1    1700 3600
@@
 F 0 "R45" V 1505 3850 50  0000 C CNN
 F 1 "2k2±5% 0.063w" V 1596 3850 50  0000 C CNN
-F 2 "" V 1630 3860 50  0000 C CNN
+F 2 "Icezum:R_0402" V 1630 3860 50  0001 C CNN
 F 3 "" H 1700 3860 50  0000 C CNN
 	1    1700 4000
@@
 F 0 "SW1" H 5000 1550 60  0000 C CNN
 F 1 "Switch" H 5000 1250 60  0000 C CNN
-F 2 "" H 4600 1350 60  0000 C CNN
+F 2 "Icezum:WE_434331013822_push_switch" H 4600 1350 60  0001 C CNN
 F 3 "" H 4600 1350 60  0000 C CNN
 	1    4600 1350
@@
 F 0 "SW2" H 5000 2450 60  0000 C CNN
 F 1 "Switch" H 5000 2150 60  0000 C CNN
-F 2 "" H 4600 2250 60  0000 C CNN
+F 2 "Icezum:WE_434331013822_push_switch" H 4600 2250 60  0001 C CNN
 F 3 "" H 4600 2250 60  0000 C CNN
 	1    4600 2250
@@
 F 0 "R31" V 4150 1650 50  0000 C CNN
 F 1 "10k±5% 0.0625w" V 4250 1700 50  0000 C CNN
-F 2 "" V 4280 1560 50  0000 C CNN
+F 2 "Icezum:R_0402" V 4280 1560 50  0001 C CNN
 F 3 "" H 4350 1560 50  0000 C CNN
 	1    4350 1700
@@
 F 0 "R32" V 4150 2550 50  0000 C CNN
 F 1 "10k±5% 0.0625w" V 4250 2600 50  0000 C CNN
-F 2 "" V 4280 2460 50  0000 C CNN
+F 2 "Icezum:R_0402" V 4280 2460 50  0001 C CNN
 F 3 "" H 4350 2460 50  0000 C CNN
 	1    4350 2600

Commit message: Colocadas todas las vias y corregir error en simbolo de pulsadores 4p
Parts:
- SW1, SW2: value Switch -> Switch_4p
Changed lines of the file:
@@
-EESchema Schematic File Version 3
+EESchema Schematic File Version 2
 LIBS:icezum
-LIBS:icezum-cache
 EELAYER 26 0
 EELAYER END
@@
 	0    1    1    0
 $EndComp
-$Comp
-L Switch_4p SW1
-U 1 1 59F1BB8D
-P 4600 1350
-F 0 "SW1" H 5000 1550 60  0000 C CNN
-F 1 "Switch" H 5000 1250 60  0000 C CNN
-F 2 "Icezum:WE_434331013822_push_switch" H 4600 1350 60  0001 C CNN
-F 3 "" H 4600 1350 60  0000 C CNN
-	1    4600 1350
-	1    0    0    -1
-$EndComp
 Wire Wire Line
 	5350 1450 5400 1450
 Connection ~ 5400 1450
-$Comp
-L Switch_4p SW2
-U 1 1 59F1C092
-P 4600 2250
-F 0 "SW2" H 5000 2450 60  0000 C CNN
-F 1 "Switch" H 5000 2150 60  0000 C CNN
-F 2 "Icezum:WE_434331013822_push_switch" H 4600 2250 60  0001 C CNN
-F 3 "" H 4600 2250 60  0000 C CNN
-	1    4600 2250
-	1    0    0    -1
-$EndComp
 Wire Wire Line
 	5400 2350 5350 2350
@@
 $EndComp
 Connection ~ 5400 1350
+$Comp
+L Switch_4p SW1
+U 1 1 59FA1B7A
+P 4600 1350
+F 0 "SW1" H 4975 1543 60  0000 C CNN
+F 1 "Switch_4p" H 4975 1543 60  0001 C CNN
+F 2 "Icezum:WE_434331013822_push_switch" H 4975 1543 60  0001 C CNN
+F 3 "" H 4600 1350 60  0000 C CNN
+	1    4600 1350
+	1    0    0    -1
+$EndComp
+$Comp
+L Switch_4p SW2
+U 1 1 59FA1F8B
+P 4600 2250
+F 0 "SW2" H 4975 2443 60  0000 C CNN
+F 1 "Switch_4p" H 4975 2443 60  0001 C CNN
+F 2 "Icezum:WE_434331013822_push_switch" H 4975 2443 60  0001 C CNN
+F 3 "" H 4600 2250 60  0000 C CNN
+	1    4600 2250
+	1    0    0    -1
+$EndComp
 $EndSCHEMATC

Commit message: importados cambios en huellas y regenerar netlist
Parts:
- SW1, SW2: symbol Switch_4p -> Switch_4p-RESCUE-icezum
- U7: footprint Icezum:QFN16 -> Icezum:QFN16_VIATP
Changed lines of the file:
@@
-EESchema Schematic File Version 2
+EESchema Schematic File Version 3
+LIBS:icezum-rescue
 LIBS:icezum
+LIBS:icezum-cache
 EELAYER 26 0
 EELAYER END
@@
 F 0 "U7" H 8470 2680 60  0000 L BNN
 F 1 "ADS7924" H 9130 2680 60  0000 L BNN
-F 2 "Icezum:QFN16" H 8470 2660 60  0001 C CNN
+F 2 "Icezum:QFN16_VIATP" H 8470 2660 60  0001 C CNN
 F 3 "" H 8470 2660 60  0000 C CNN
 	1    8250 2550
@@
 Connection ~ 5400 1350
 $Comp
-L Switch_4p SW1
+L Switch_4p-RESCUE-icezum SW1
 U 1 1 59FA1B7A
 P 4600 1350
+AR Path="/59FA1B7A" Ref="SW1"  Part="1"
+AR Path="/57489FE9/59FA1B7A" Ref="SW1"  Part="1"
 F 0 "SW1" H 4975 1543 60  0000 C CNN
 F 1 "Switch_4p" H 4975 1543 60  0001 C CNN
@@
 $EndComp
 $Comp
-L Switch_4p SW2
+L Switch_4p-RESCUE-icezum SW2
 U 1 1 59FA1F8B
 P 4600 2250
+AR Path="/59FA1F8B" Ref="SW2"  Part="1"
+AR Path="/57489FE9/59FA1F8B" Ref="SW2"  Part="1"
 F 0 "SW2" H 4975 2443 60  0000 C CNN
 F 1 "Switch_4p" H 4975 2443 60  0001 C CNN

Commit message: se cambia el nombre de la huella para los pulsadores y se actualiza en esquema y netlist
Parts:
- SW1, SW2: footprint Icezum:WE_434331013822_push_switch -> Icezum:WE_434331013822
Changed lines of the file:
@@
 F 0 "SW1" H 4975 1543 60  0000 C CNN
 F 1 "Switch_4p" H 4975 1543 60  0001 C CNN
-F 2 "Icezum:WE_434331013822_push_switch" H 4975 1543 60  0001 C CNN
+F 2 "Icezum:WE_434331013822" H 4975 1543 60  0001 C CNN
 F 3 "" H 4600 1350 60  0000 C CNN
 	1    4600 1350
@@
 F 0 "SW2" H 4975 2443 60  0000 C CNN
 F 1 "Switch_4p" H 4975 2443 60  0001 C CNN
-F 2 "Icezum:WE_434331013822_push_switch" H 4975 2443 60  0001 C CNN
+F 2 "Icezum:WE_434331013822" H 4975 2443 60  0001 C CNN
 F 3 "" H 4600 2250 60  0000 C CNN
 	1    4600 2250

Commit message: Symbol library updated to the latest kicad
Parts:
- C34, C35, C41, C45, C46: symbol C -> icezum:C
- DOC3: symbol icezum-headers-doc -> icezum:icezum-headers-doc
- DOC4, DOC5: symbol switch_DOC -> icezum:switch_DOC
- J15, J16, J17: symbol 1x4_male_pin_Header_2.54mm -> icezum:1x4_male_pin_Header_2.54mm
- JP1: symbol Jumper_3pin -> icezum:Jumper_3pin
- JPM1: symbol Jumper_1x2_Mech -> icezum:Jumper_1x2_Mech
- LD0, LD1, LD2, LD3, LD4, LD5, LD6, LD7: symbol LED -> icezum:LED
- R17, R18, R19, R20, R21, R31, R32, R40, R41, R42, R43, R44, R45: symbol R -> icezum:R
- U7: symbol ADS7924 -> icezum:ADS7924
- doc10: symbol 1x3_pin_male_header_v_DOC -> icezum:1x3_pin_male_header_v_DOC
- doc9: symbol 3x4_pin_male_header_DOC -> icezum:3x4_pin_male_header_DOC
Changed lines of the file:
@@
-EESchema Schematic File Version 3
-LIBS:icezum-rescue
-LIBS:icezum
+EESchema Schematic File Version 4
 LIBS:icezum-cache
 EELAYER 26 0
@@
 $EndDescr
 $Comp
-L icezum-headers-doc DOC3
+L icezum:icezum-headers-doc DOC3
 U 1 1 5748B0A8
 P 3500 6650
@@
 $EndComp
 $Comp
-L ADS7924 U7
+L icezum:ADS7924 U7
 U 1 1 5748BFE4
 P 8250 2550
@@
 $EndComp
 $Comp
-L Jumper_3pin JP1
+L icezum:Jumper_3pin JP1
 U 1 1 5748CA2F
 P 7350 1550
@@
 $EndComp
 $Comp
-L +5V #PWR0111
+L icezum:+5V #PWR0111
 U 1 1 5748CB4A
 P 7350 1450
@@
 AREF
 $Comp
-L C C41
+L icezum:C C41
 U 1 1 5748E340
 P 8600 1650
@@
 $EndComp
 $Comp
-L R R19
+L icezum:R R19
 U 1 1 5748E354
 P 7900 2050
@@
 $EndComp
 $Comp
-L C C46
+L icezum:C C46
 U 1 1 574908C6
 P 8600 2050
@@
 $EndComp
 $Comp
-L GNDREF #PWR0112
+L icezum:GNDREF #PWR0112
 U 1 1 57491733
 P 9000 2150
@@
 $EndComp
 $Comp
-L C C45
+L icezum:C C45
 U 1 1 57491D8E
 P 9400 2050
@@
 $EndComp
 $Comp
-L +3V3 #PWR0113
+L icezum:+3V3 #PWR0113
 U 1 1 574923BF
 P 9850 1650
@@
 $EndComp
 $Comp
-L R R20
+L icezum:R R20
 U 1 1 5749366D
 P 10050 2500
@@
 $EndComp
 $Comp
-L R R21
+L icezum:R R21
 U 1 1 57493DA0
 P 10300 2500
@@
 NoConn ~ 9800 3350
 $Comp
-L GNDREF #PWR0114
+L icezum:GNDREF #PWR0114
 U 1 1 5749574F
 P 9900 3750
@@
 $EndComp
 $Comp
-L GNDREF #PWR0115
+L icezum:GNDREF #PWR0115
 U 1 1 57495E07
 P 8200 3750
@@
 $EndComp
 $Comp
-L 1x4_male_pin_Header_2.54mm J17
+L icezum:1x4_male_pin_Header_2.54mm J17
 U 1 1 57497491
 P 7900 3100
@@
 A3
 $Comp
-L 3x4_pin_male_header_DOC doc9
+L icezum:3x4_pin_male_header_DOC doc9
 U 1 1 5749A2B2
 P 7550 4650
@@
 $EndComp
 $Comp
-L 1x4_male_pin_Header_2.54mm J15
+L icezum:1x4_male_pin_Header_2.54mm J15
 U 1 1 5749B012
 P 7350 3100
@@
 $EndComp
 $Comp
-L +5V_P #PWR0116
+L icezum:+5V_P #PWR0116
 U 1 1 5749B123
 P 7400 2850
@@
 A0
 $Comp
-L 1x4_male_pin_Header_2.54mm J16
+L icezum:1x4_male_pin_Header_2.54mm J16
 U 1 1 5749ECA7
 P 6850 3100
@@
 1x4 male pin header 2.54mm
 $Comp
-L GNDREF #PWR0117
+L icezum:GNDREF #PWR0117
 U 1 1 5749ED8F
 P 6900 3550
@@
 4-Channel I2C ADC
 $Comp
-L Jumper_1x2_Mech JPM1
+L icezum:Jumper_1x2_Mech JPM1
 U 1 1 574A0E14
 P 7450 1000
@@
 $EndComp
 $Comp
-L 1x3_pin_male_header_v_DOC doc10
+L icezum:1x3_pin_male_header_v_DOC doc10
 U 1 1 574A23B9
 P 8250 1100
@@
 AREF
 $Comp
-L LED LD0
+L icezum:LED LD0
 U 1 1 574A356F
 P 1950 1200
@@
 LED0
 $Comp
-L LED LD1
+L icezum:LED LD1
 U 1 1 574A6DB7
 P 1950 1600
@@
 LED1
 $Comp
-L LED LD2
+L icezum:LED LD2
 U 1 1 574A7937
 P 1950 2000
@@
 LED2
 $Comp
-L LED LD3
+L icezum:LED LD3
 U 1 1 574A81AF
 P 1950 2400
@@
 LED3
 $Comp
-L LED LD4
+L icezum:LED LD4
 U 1 1 574A8C2D
 P 1950 2800
@@
 LED4
 $Comp
-L LED LD5
+L icezum:LED LD5
 U 1 1 574A8C3C
 P 1950 3200
@@
 LED5
 $Comp
-L LED LD6
+L icezum:LED LD6
 U 1 1 574A8C4B
 P 1950 3600
@@
 LED6
 $Comp
-L LED LD7
+L icezum:LED LD7
 U 1 1 574A8C5A
 P 1950 4000
@@
 LED7
 $Comp
-L GNDREF #PWR0118
+L icezum:GNDREF #PWR0118
 U 1 1 574AA29A
 P 2750 4200
@@
 	3300 4500 3300 500
 $Comp
-L C C34
+L icezum:C C34
 U 1 1 574AD7AC
 P 3950 1600
@@
 	3950 1350 3950 1450
 $Comp
-L GNDREF #PWR0119
+L icezum:GNDREF #PWR0119
 U 1 1 574AFC1C
 P 3950 1800
@@
 User Switches
 $Comp
-L C C35
+L icezum:C C35
 U 1 1 574B168A
 P 3950 2500
@@
 	3950 2250 3950 2350
 $Comp
-L GNDREF #PWR0121
+L icezum:GNDREF #PWR0121
 U 1 1 574B1692
 P 3950 2700
@@
 Connection ~ 3950 2250
 $Comp
-L switch_DOC DOC4
+L icezum:switch_DOC DOC4
 U 1 1 574B2283
 P 5650 1450
@@
 $EndComp
 $Comp
-L switch_DOC DOC5
+L icezum:switch_DOC DOC5
 U 1 1 574B2315
 P 5650 2350
@@
 $EndBitmap
 $Comp
-L GNDREF #PWR0123
+L icezum:GNDREF #PWR0123
 U 1 1 57802053
 P 9000 3950
@@
 $EndComp
 $Comp
-L R R18
+L icezum:R R18
 U 1 1 59F17BE6
 P 1700 1600
@@
 $EndComp
 $Comp
-L R R17
+L icezum:R R17
 U 1 1 59F17E30
 P 1700 1200
@@
 $EndComp
 $Comp
-L R R40
+L icezum:R R40
 U 1 1 59F18019
 P 1700 2000
@@
 $EndComp
 $Comp
-L R R41
+L icezum:R R41
 U 1 1 59F1806F
 P 1700 2400
@@
 $EndComp
 $Comp
-L R R42
+L icezum:R R42
 U 1 1 59F180C7
 P 1700 2800
@@
 $EndComp
 $Comp
-L R R43
+L icezum:R R43
 U 1 1 59F18121
 P 1700 3200
@@
 $EndComp
 $Comp
-L R R44
+L icezum:R R44
 U 1 1 59F181DC
 P 1700 3600
@@
 $EndComp
 $Comp
-L R R45
+L icezum:R R45
 U 1 1 59F18236
 P 1700 4000
@@
 Connection ~ 4550 2250
 $Comp
-L R R31
+L icezum:R R31
 U 1 1 59F1CA9F
 P 4350 1700
@@
 $EndComp
 $Comp
-L GNDREF #PWR099
+L icezum:GNDREF #PWR099
 U 1 1 59F1CE1A
 P 4350 1800
@@
 Connection ~ 4350 1350
 $Comp
-L R R32
+L icezum:R R32
 U 1 1 59F1D353
 P 4350 2600
@@
 $EndComp
 $Comp
-L GNDREF #PWR0105
+L icezum:GNDREF #PWR0105
 U 1 1 59F1D35A
 P 4350 2700
@@
 Connection ~ 4350 2250
 $Comp
-L +3V3 #PWR0120
+L icezum:+3V3 #PWR0120
 U 1 1 59F1D584
 P 5400 1150
