File: src-kicad/arduino-sockets.sch (KiCad schematic (older format))
At the start: 48 parts, among them J10 1x8_female_pin_Header_2.54mm, J11 1x6_female_pin_Header_2.54mm, J12 1x6_male_pin_Header_2.54mm, J13 1x6_male_pin_Header_2.54mm, J14 1x6_male_pin_Header_2.54mm, J19 2x4_male_pin_Header_2.54mm, J2 1x6_male_pin_Header_2.54mm, J3 1x6_male_pin_Header_2.54mm, J4 1x10_female_pin_Header_2.54mm, J5 1x8_female_pin_Header_2.54mm, J6 1x6_male_pin_Header_2.54mm, J7 1x8_male_pin_Header_2.54mm, J8 1x8_male_pin_Header_2.54mm, J9 1x8_male_pin_Header_2.54mm, U6 TXB0106, U8 TXS0108, U9 TXB0108

Commit message: Kicad pcb migration: Capacitors C21, C26 and C30
Parts:
- C36, C37, C47, C48, C49, C50: footprint (none) -> Icezum:C_0402
Changed lines of the file:
@@
 F 0 "C49" V 1100 5650 50  0000 L CNN
 F 1 "100nF" V 1200 5650 50  0000 L CNN
-F 2 "" H 1388 5600 50  0000 C CNN
+F 2 "Icezum:C_0402" H 1388 5600 50  0001 C CNN
 F 3 "" H 1350 5750 50  0000 C CNN
 F 4 "X7R" V 1420 5620 50  0000 C CNN "Class"
@@
 F 0 "C50" V 1800 5650 50  0000 L CNN
 F 1 "100nF" V 1900 5650 50  0000 L CNN
-F 2 "" H 2088 5600 50  0000 C CNN
+F 2 "Icezum:C_0402" H 2088 5600 50  0001 C CNN
 F 3 "" H 2050 5750 50  0000 C CNN
 F 4 "X7R" V 2120 5620 50  0000 C CNN "Class"
@@
 F 0 "C36" V 1200 3300 50  0000 L CNN
 F 1 "100nF" V 1300 3050 50  0000 L CNN
-F 2 "" H 1388 3200 50  0000 C CNN
+F 2 "Icezum:C_0402" H 1388 3200 50  0001 C CNN
 F 3 "" H 1350 3350 50  0000 C CNN
 F 4 "X7R" V 1420 3220 50  0000 C CNN "Class"
@@
 F 0 "C37" V 1900 3250 50  0000 L CNN
 F 1 "100nF" V 2000 3050 50  0000 L CNN
-F 2 "" H 2088 3200 50  0000 C CNN
+F 2 "Icezum:C_0402" H 2088 3200 50  0001 C CNN
 F 3 "" H 2050 3350 50  0000 C CNN
 F 4 "X7R" V 2120 3220 50  0000 C CNN "Class"
@@
 F 0 "C47" V 1200 850 50  0000 L CNN
 F 1 "100nF" V 1300 850 50  0000 L CNN
-F 2 "" H 1488 800 50  0000 C CNN
+F 2 "Icezum:C_0402" H 1488 800 50  0001 C CNN
 F 3 "" H 1450 950 50  0000 C CNN
 F 4 "X7R" V 1520 820 50  0000 C CNN "Class"
@@
 F 0 "C48" V 1900 850 50  0000 L CNN
 F 1 "100nF" V 2000 850 50  0000 L CNN
-F 2 "" H 2188 800 50  0000 C CNN
+F 2 "Icezum:C_0402" H 2188 800 50  0001 C CNN
 F 3 "" H 2150 950 50  0000 C CNN
 F 4 "X7R" V 2220 820 50  0000 C CNN "Class"
@@
 B8 D2 A5 D0 D0 88 43 83 08 6C BD D2 A5 D0 D0 88 C3 36 11 89 E7 80 EE 2B 5D 12 0D 8D 28 1C 42 E0
 0D 11 99 76 E0 6E E0 E3 2B 5D 22 0D 8D 71 EC 07 1E E7 1B 7C F8 FF 01 FB D1 C8 6E 4C 03 14 F4 00
-00 00 00 49 45 4E 44 AE 42 60 82 00
+00 00 00 49 45 4E 44 AE 42 60 82 03
 EndData
 $EndBitmap

Commit message: Kicad pcb migration: More capacitors footprint assigned
Parts:
- C38, C39, C40, C42, C43, C44, C51, C52, C53, C54, C55, C56, C57, C58: footprint (none) -> Icezum:C_0402
Changed lines of the file:
@@
 F 0 "C54" H 2310 7550 50  0000 L CNN
 F 1 "100pF" H 2310 7480 50  0000 L CNN
-F 2 "" H 2338 7250 50  0000 C CNN
+F 2 "Icezum:C_0402" H 2338 7250 50  0001 C CNN
 F 3 "" H 2300 7400 50  0000 C CNN
 F 4 "X7R" H 2400 7300 50  0000 C CNN "Class"
@@
 F 0 "C55" H 2610 7550 50  0000 L CNN
 F 1 "100pF" H 2610 7480 50  0000 L CNN
-F 2 "" H 2638 7250 50  0000 C CNN
+F 2 "Icezum:C_0402" H 2638 7250 50  0001 C CNN
 F 3 "" H 2600 7400 50  0000 C CNN
 F 4 "X7R" H 2700 7300 50  0000 C CNN "Class"
@@
 F 0 "C51" H 2910 7350 50  0000 L CNN
 F 1 "100pF" H 2910 7280 50  0000 L CNN
-F 2 "" H 2938 7050 50  0000 C CNN
+F 2 "Icezum:C_0402" H 2938 7050 50  0001 C CNN
 F 3 "" H 2900 7200 50  0000 C CNN
 F 4 "X7R" H 3000 7100 50  0000 C CNN "Class"
@@
 F 0 "C56" H 3210 7550 50  0000 L CNN
 F 1 "100pF" H 3210 7480 50  0000 L CNN
-F 2 "" H 3238 7250 50  0000 C CNN
+F 2 "Icezum:C_0402" H 3238 7250 50  0001 C CNN
 F 3 "" H 3200 7400 50  0000 C CNN
 F 4 "X7R" H 3300 7300 50  0000 C CNN "Class"
@@
 F 0 "C52" H 3510 7250 50  0000 L CNN
 F 1 "100pF" H 3510 7180 50  0000 L CNN
-F 2 "" H 3538 6950 50  0000 C CNN
+F 2 "Icezum:C_0402" H 3538 6950 50  0001 C CNN
 F 3 "" H 3500 7100 50  0000 C CNN
 F 4 "X7R" H 3600 7000 50  0000 C CNN "Class"
@@
 F 0 "C57" H 3810 7550 50  0000 L CNN
 F 1 "100pF" H 3810 7480 50  0000 L CNN
-F 2 "" H 3838 7250 50  0000 C CNN
+F 2 "Icezum:C_0402" H 3838 7250 50  0000 C CNN
 F 3 "" H 3800 7400 50  0000 C CNN
 F 4 "X7R" H 3900 7300 50  0000 C CNN "Class"
@@
 F 0 "C53" H 4110 7250 50  0000 L CNN
 F 1 "100pF" H 4110 7180 50  0000 L CNN
-F 2 "" H 4138 6950 50  0000 C CNN
+F 2 "Icezum:C_0402" H 4138 6950 50  0001 C CNN
 F 3 "" H 4100 7100 50  0000 C CNN
 F 4 "X7R" H 4200 7000 50  0000 C CNN "Class"
@@
 F 0 "C58" H 4410 7550 50  0000 L CNN
 F 1 "100pF" H 4410 7480 50  0000 L CNN
-F 2 "" H 4438 7250 50  0000 C CNN
+F 2 "Icezum:C_0402" H 4438 7250 50  0001 C CNN
 F 3 "" H 4400 7400 50  0000 C CNN
 F 4 "X7R" H 4500 7300 50  0000 C CNN "Class"
@@
 F 0 "C40" H 2360 4950 50  0000 L CNN
 F 1 "100pF" H 2360 4880 50  0000 L CNN
-F 2 "" H 2388 4650 50  0000 C CNN
+F 2 "Icezum:C_0402" H 2388 4650 50  0001 C CNN
 F 3 "" H 2350 4800 50  0000 C CNN
 F 4 "X7R" H 2450 4700 50  0000 C CNN "Class"
@@
 F 0 "C42" H 2660 4950 50  0000 L CNN
 F 1 "100pF" H 2660 4880 50  0000 L CNN
-F 2 "" H 2688 4650 50  0000 C CNN
+F 2 "Icezum:C_0402" H 2688 4650 50  0001 C CNN
 F 3 "" H 2650 4800 50  0000 C CNN
 F 4 "X7R" H 2750 4700 50  0000 C CNN "Class"
@@
 F 0 "C38" H 2960 4700 50  0000 L CNN
 F 1 "100pF" H 2960 4630 50  0000 L CNN
-F 2 "" H 2988 4400 50  0000 C CNN
+F 2 "Icezum:C_0402" H 2988 4400 50  0001 C CNN
 F 3 "" H 2950 4550 50  0000 C CNN
 F 4 "X7R" H 3050 4450 50  0000 C CNN "Class"
@@
 F 0 "C43" H 3260 4950 50  0000 L CNN
 F 1 "100pF" H 3260 4880 50  0000 L CNN
-F 2 "" H 3288 4650 50  0000 C CNN
+F 2 "Icezum:C_0402" H 3288 4650 50  0001 C CNN
 F 3 "" H 3250 4800 50  0000 C CNN
 F 4 "X7R" H 3350 4700 50  0000 C CNN "Class"
@@
 F 0 "C39" H 3560 4700 50  0000 L CNN
 F 1 "100pF" H 3560 4630 50  0000 L CNN
-F 2 "" H 3588 4400 50  0000 C CNN
+F 2 "Icezum:C_0402" H 3588 4400 50  0001 C CNN
 F 3 "" H 3550 4550 50  0000 C CNN
 F 4 "X7R" H 3650 4450 50  0000 C CNN "Class"
@@
 F 0 "C44" H 3860 4950 50  0000 L CNN
 F 1 "100pF" H 3860 4880 50  0000 L CNN
-F 2 "" H 3888 4650 50  0000 C CNN
+F 2 "Icezum:C_0402" H 3888 4650 50  0001 C CNN
 F 3 "" H 3850 4800 50  0000 C CNN
 F 4 "X7R" H 3950 4700 50  0000 C CNN "Class"

Commit message: Kicad pcb migration. R11 added. Some bug fixed in the schematics (R16 was missing)
Parts:
- R22, R23: footprint (none) -> Icezum:R_0402
Changed lines of the file:
@@
 F 0 "R22" H 2480 1290 50  0000 C CNN
 F 1 "4K7±5% 0.063w" V 2670 1350 39  0000 C CNN
-F 2 "" V 2530 1450 50  0000 C CNN
+F 2 "Icezum:R_0402" V 2530 1450 50  0001 C CNN
 F 3 "" H 2600 1450 50  0000 C CNN
 	1    2600 1450
@@
 F 0 "R23" H 2880 1290 50  0000 C CNN
 F 1 "4K7±5% 0.063w" V 3070 1350 39  0000 C CNN
-F 2 "" V 2930 1450 50  0000 C CNN
+F 2 "Icezum:R_0402" V 2930 1450 50  0001 C CNN
 F 3 "" H 3000 1450 50  0000 C CNN
 	1    3000 1450
@@
 F3 F0 1D 79 17 0B BC D0 AE 96 03 B8 3F 0C 6D B8 A2 A8 0B 16 2C 58 B0 60 C1 82 05 0B 16 2C 58 B0
 60 C1 82 05 0B 16 2C 58 B0 E0 7F 81 FF 00 64 C5 01 8A 14 5C 86 66 00 00 00 00 49 45 4E 44 AE 42
-60 82 20
+60 82 39
 EndData
 $EndBitmap
